File: motherboard/motherboard.sch (EAGLE design)
At the start: 4 parts, among them U1 LED_100V_BUCK, U2 LED_100V_BUCK, U3 LED_100V_BUCK, U4 LED_100V_BUCK

Commit message: Getting started.
Parts:
- added S1: (no value), SparkFun-Electromechanical:TAC_SWITCHPTH
- added U$1: MBED_NXP_LPC1768, SparkFun-DigitalIC:MBED_NXP_LPC1768
- added U$2: OSHW-LOGOL, SparkFun-Aesthetics:OSHW-LOGOL
Connections:
- new net GND: S1.1, S1.2, U$1.P$1, U1.GND, U2.GND, U3.GND, U4.GND
- new net N$1: S1.3, S1.4, U$1.P$3
- new net V+: U1.V+, U2.V+, U3.V+
- new net VCC: U$1.P$2
Changed lines of the file:
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@@
 <layer number="48" name="Document" color="7" fill="1" visible="no" active="no"/>
 <layer number="49" name="Reference" color="7" fill="1" visible="no" active="no"/>
+<layer number="50" name="dxf" color="7" fill="1" visible="no" active="no"/>
 <layer number="51" name="tDocu" color="7" fill="1" visible="no" active="no"/>
 <layer number="52" name="bDocu" color="7" fill="1" visible="no" active="no"/>
+<layer number="53" name="tGND_GNDA" color="7" fill="9" visible="no" active="no"/>
+<layer number="54" name="bGND_GNDA" color="1" fill="9" visible="no" active="no"/>
+<layer number="56" name="wert" color="7" fill="1" visible="no" active="no"/>
 <layer number="91" name="Nets" color="2" fill="1" visible="yes" active="yes"/>
 <layer number="92" name="Busses" color="1" fill="1" visible="yes" active="yes"/>
@@
 <layer number="97" name="Info" color="7" fill="1" visible="yes" active="yes"/>
 <layer number="98" name="Guide" color="6" fill="1" visible="yes" active="yes"/>
+<layer number="100" name="Muster" color="7" fill="1" visible="no" active="no"/>
+<layer number="101" name="Patch_Top" color="12" fill="4" visible="no" active="yes"/>
+<layer number="102" name="Vscore" color="7" fill="1" visible="no" active="yes"/>
+<layer number="103" name="tMap" color="7" fill="1" visible="no" active="yes"/>
+<layer number="104" name="Name" color="16" fill="1" visible="no" active="yes"/>
+<layer number="105" name="tPlate" color="7" fill="1" visible="no" active="yes"/>
+<layer number="106" name="bPlate" color="7" fill="1" visible="no" active="yes"/>
+<layer number="107" name="Crop" color="7" fill="1" visible="no" active="yes"/>
+<layer number="116" name="Patch_BOT" color="9" fill="4" visible="no" active="yes"/>
+<layer number="121" name="_tsilk" color="7" fill="1" visible="no" active="yes"/>
+<layer number="122" name="_bsilk" color="7" fill="1" visible="no" active="yes"/>
+<layer number="125" name="_tNames" color="7" fill="1" visible="no" active="yes"/>
+<layer number="144" name="Drill_legend" color="7" fill="1" visible="no" active="yes"/>
+<layer number="151" name="HeatSink" color="7" fill="1" visible="no" active="yes"/>
+<layer number="199" name="Contour" color="7" fill="1" visible="yes" active="yes"/>
+<layer number="200" name="200bmp" color="1" fill="10" visible="no" active="yes"/>
+<layer number="201" name="201bmp" color="2" fill="10" visible="no" active="yes"/>
+<layer number="202" name="202bmp" color="3" fill="10" visible="no" active="yes"/>
+<layer number="203" name="203bmp" color="4" fill="10" visible="no" active="yes"/>
+<layer number="204" name="204bmp" color="5" fill="10" visible="no" active="yes"/>
+<layer number="205" name="205bmp" color="6" fill="10" visible="no" active="yes"/>
+<layer number="206" name="206bmp" color="7" fill="10" visible="no" active="yes"/>
+<layer number="207" name="207bmp" color="8" fill="10" visible="no" active="yes"/>
+<layer number="208" name="208bmp" color="9" fill="10" visible="no" active="yes"/>
+<layer number="209" name="209bmp" color="7" fill="1" visible="no" active="yes"/>
+<layer number="210" name="210bmp" color="7" fill="1" visible="no" active="yes"/>
+<layer number="211" name="211bmp" color="7" fill="1" visible="no" active="yes"/>
+<layer number="212" name="212bmp" color="7" fill="1" visible="no" active="yes"/>
+<layer number="213" name="213bmp" color="7" fill="1" visible="no" active="yes"/>
+<layer number="214" name="214bmp" color="7" fill="1" visible="no" active="yes"/>
+<layer number="215" name="215bmp" color="7" fill="1" visible="no" active="yes"/>
+<layer number="216" name="216bmp" color="7" fill="1" visible="no" active="yes"/>
+<layer number="217" name="217bmp" color="18" fill="1" visible="no" active="no"/>
+<layer number="218" name="218bmp" color="19" fill="1" visible="no" active="no"/>
+<layer number="219" name="219bmp" color="20" fill="1" visible="no" active="no"/>
+<layer number="220" name="220bmp" color="21" fill="1" visible="no" active="no"/>
+<layer number="221" name="221bmp" color="22" fill="1" visible="no" active="no"/>
+<layer number="222" name="222bmp" color="23" fill="1" visible="no" active="no"/>
+<layer number="223" name="223bmp" color="24" fill="1" visible="no" active="no"/>
+<layer number="224" name="224bmp" color="25" fill="1" visible="no" active="no"/>
+<layer number="250" name="Descript" color="3" fill="1" visible="no" active="no"/>
+<layer number="251" name="SMDround" color="12" fill="11" visible="no" active="no"/>
+<layer number="254" name="cooling" color="7" fill="1" visible="no" active="yes"/>
 </layers>
 <schematic xreflabel="%F%N/%S.%C%R" xrefpart="/%S.%C%R">
@@
 <part name="U3" library="LED-drivers" deviceset="LED_100V_BUCK" device=""/>
 <part name="U4" library="LED-drivers" deviceset="LED_100V_BUCK" device=""/>
+<part name="U$1" library="SparkFun-DigitalIC" deviceset="MBED_NXP_LPC1768" device=""/>
+<part name="GND1" library="supply1" deviceset="GND" device=""/>
+<part name="P+1" library="supply1" deviceset="VCC" device=""/>
+<part name="U$2" library="SparkFun-Aesthetics" deviceset="OSHW-LOGO" device="L"/>
+<part name="S1" library="SparkFun-Electromechanical" deviceset="TAC_SWITCH" device="PTH"/>
+<part name="GND2" library="supply1" deviceset="GND" device=""/>
+<part name="P+2" library="supply1" deviceset="V+" device=""/>
+<part name="P+3" library="supply1" deviceset="V+" device=""/>
+<part name="P+4" library="supply1" deviceset="V+" device=""/>
+<part name="GND3" library="supply1" deviceset="GND" device=""/>
+<part name="GND4" library="supply1" deviceset="GND" device=""/>
+<part name="GND5" library="supply1" deviceset="GND" device=""/>
+<part name="GND6" library="supply1" deviceset="GND" device=""/>
 </parts>
 <sheets>
@@
 <instance part="U3" gate="G$1" x="226.06" y="55.88"/>
 <instance part="U4" gate="G$1" x="307.34" y="53.34"/>
+<instance part="U$1" gate="G$1" x="-5.08" y="269.24"/>
+<instance part="GND1" gate="1" x="-50.8" y="292.1" rot="R270"/>
+<instance part="P+1" gate="VCC" x="-50.8" y="289.56" rot="R90"/>
+<instance part="U$2" gate="G$1" x="0" y="2.54"/>
+<instance part="S1" gate="S" x="-68.58" y="289.56"/>
+<instance part="GND2" gate="1" x="-73.66" y="284.48"/>
+<instance part="P+2" gate="1" x="38.1" y="83.82"/>
+<instance part="P+3" gate="1" x="142.24" y="83.82"/>
+<instance part="P+4" gate="1" x="226.06" y="86.36"/>
+<instance part="GND3" gate="1" x="38.1" y="22.86"/>
+<instance part="GND4" gate="1" x="142.24" y="22.86"/>
+<instance part="GND5" gate="1" x="226.06" y="25.4"/>
+<instance part="GND6" gate="1" x="307.34" y="22.86"/>
 </instances>
 <busses>
 </busses>
 <nets>
+<net name="GND" class="0">
+<segment>
+<pinref part="U$1" gate="G$1" pin="P$1"/>
+<pinref part="GND1" gate="1" pin="GND"/>
+<wire x1="-48.26" y1="292.1" x2="-38.1" y2="292.1" width="0.1524" layer="91"/>
+</segment>
+<segment>
+<pinref part="S1" gate="S" pin="2"/>
+<pinref part="GND2" gate="1" pin="GND"/>
+<pinref part="S1" gate="S" pin="1"/>
+<wire x1="-73.66" y1="287.02" x2="-73.66" y2="289.56" width="0.1524" layer="91"/>
+<junction x="-73.66" y="287.02"/>
+</segment>
+<segment>
+<pinref part="U1" gate="G$1" pin="GND"/>
+<pinref part="GND3" gate="1" pin="GND"/>
+</segment>
+<segment>
+<pinref part="U2" gate="G$1" pin="GND"/>
+<pinref part="GND4" gate="1" pin="GND"/>
+</segment>
+<segment>
+<pinref part="U3" gate="G$1" pin="GND"/>
+<pinref part="GND5" gate="1" pin="GND"/>
+</segment>
+<segment>
+<pinref part="U4" gate="G$1" pin="GND"/>
+<pinref part="GND6" gate="1" pin="GND"/>
+</segment>
+</net>
+<net name="VCC" class="0">
+<segment>
+<pinref part="U$1" gate="G$1" pin="P$2"/>
+<pinref part="P+1" gate="VCC" pin="VCC"/>
+<wire x1="-48.26" y1="289.56" x2="-38.1" y2="289.56" width="0.1524" layer="91"/>
+</segment>
+</net>
+<net name="N$1" class="0">
+<segment>
+<pinref part="U$1" gate="G$1" pin="P$3"/>
+<pinref part="S1" gate="S" pin="4"/>
+<wire x1="-38.1" y1="287.02" x2="-63.5" y2="287.02" width="0.1524" layer="91"/>
+<pinref part="S1" gate="S" pin="3"/>
+<wire x1="-63.5" y1="287.02" x2="-63.5" y2="289.56" width="0.1524" layer="91"/>
+<junction x="-63.5" y="287.02"/>
+</segment>
+</net>
+<net name="V+" class="0">
+<segment>
+<pinref part="U1" gate="G$1" pin="V+"/>
+<pinref part="P+2" gate="1" pin="V+"/>
+</segment>
+<segment>
+<pinref part="U2" gate="G$1" pin="V+"/>
+<pinref part="P+3" gate="1" pin="V+"/>
+</segment>
+<segment>
+<pinref part="U3" gate="G$1" pin="V+"/>
+<pinref part="P+4" gate="1" pin="V+"/>
+</segment>
+</net>
 </nets>
 </sheet>

Commit message: incremental progress
Parts:
- added U$3: M04X2, SparkFun-Connectors:M04X2
Connections:
- net VCC renamed +5V
- new net +3V3: U$1.P$40
- new net N$2: U$3.1, U1.LED_C
- new net N$3: U$3.3, U2.LED_C
- new net N$4: U$3.5, U3.LED_C
- new net N$5: U$3.7, U4.LED_C
- new net N$6: U$3.2, U1.LED_A
- new net N$7: U$3.4, U2.LED_A
- new net N$8: U$3.6, U3.LED_A
- new net N$9: U$3.8, U4.LED_A
- net V+: now also U4.V+
Other:
- moved on the sheet: U2, U3, U4
Changed lines of the file:
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@@
 <part name="U$1" library="SparkFun-DigitalIC" deviceset="MBED_NXP_LPC1768" device=""/>
 <part name="GND1" library="supply1" deviceset="GND" device=""/>
-<part name="P+1" library="supply1" deviceset="VCC" device=""/>
 <part name="U$2" library="SparkFun-Aesthetics" deviceset="OSHW-LOGO" device="L"/>
 <part name="S1" library="SparkFun-Electromechanical" deviceset="TAC_SWITCH" device="PTH"/>
@@
 <part name="GND5" library="supply1" deviceset="GND" device=""/>
 <part name="GND6" library="supply1" deviceset="GND" device=""/>
+<part name="P+5" library="supply1" deviceset="V+" device=""/>
+<part name="U$3" library="SparkFun-Connectors" deviceset="M04X2" device=""/>
+<part name="+3V1" library="supply1" deviceset="+3V3" device=""/>
+<part name="P+6" library="supply1" deviceset="+5V" device=""/>
 </parts>
 <sheets>
@@
 <instances>
 <instance part="U1" gate="G$1" x="38.1" y="53.34"/>
-<instance part="U2" gate="G$1" x="142.24" y="53.34"/>
-<instance part="U3" gate="G$1" x="226.06" y="55.88"/>
-<instance part="U4" gate="G$1" x="307.34" y="53.34"/>
+<instance part="U2" gate="G$1" x="96.52" y="53.34"/>
+<instance part="U3" gate="G$1" x="154.94" y="53.34"/>
+<instance part="U4" gate="G$1" x="210.82" y="53.34"/>
 <instance part="U$1" gate="G$1" x="-5.08" y="269.24"/>
 <instance part="GND1" gate="1" x="-50.8" y="292.1" rot="R270"/>
-<instance part="P+1" gate="VCC" x="-50.8" y="289.56" rot="R90"/>
 <instance part="U$2" gate="G$1" x="0" y="2.54"/>
 <instance part="S1" gate="S" x="-68.58" y="289.56"/>
 <instance part="GND2" gate="1" x="-73.66" y="284.48"/>
 <instance part="P+2" gate="1" x="38.1" y="83.82"/>
-<instance part="P+3" gate="1" x="142.24" y="83.82"/>
-<instance part="P+4" gate="1" x="226.06" y="86.36"/>
+<instance part="P+3" gate="1" x="96.52" y="83.82"/>
+<instance part="P+4" gate="1" x="154.94" y="83.82"/>
 <instance part="GND3" gate="1" x="38.1" y="22.86"/>
-<instance part="GND4" gate="1" x="142.24" y="22.86"/>
-<instance part="GND5" gate="1" x="226.06" y="25.4"/>
-<instance part="GND6" gate="1" x="307.34" y="22.86"/>
+<instance part="GND4" gate="1" x="96.52" y="22.86"/>
+<instance part="GND5" gate="1" x="154.94" y="22.86"/>
+<instance part="GND6" gate="1" x="210.82" y="22.86"/>
+<instance part="P+5" gate="1" x="210.82" y="83.82"/>
+<instance part="U$3" gate="G$1" x="254" y="-5.08" rot="R90"/>
+<instance part="+3V1" gate="G$1" x="43.18" y="292.1" rot="R270"/>
+<instance part="P+6" gate="1" x="-50.8" y="289.56" rot="R90"/>
 </instances>
 <busses>
@@
 </segment>
 </net>
-<net name="VCC" class="0">
-<segment>
-<pinref part="U$1" gate="G$1" pin="P$2"/>
-<pinref part="P+1" gate="VCC" pin="VCC"/>
-<wire x1="-48.26" y1="289.56" x2="-38.1" y2="289.56" width="0.1524" layer="91"/>
-</segment>
-</net>
 <net name="N$1" class="0">
 <segment>
@@
 <pinref part="P+4" gate="1" pin="V+"/>
 </segment>
+<segment>
+<pinref part="U4" gate="G$1" pin="V+"/>
+<pinref part="P+5" gate="1" pin="V+"/>
+</segment>
 </net>
+<net name="N$2" class="0">
+<segment>
+<pinref part="U1" gate="G$1" pin="LED_C"/>
+<wire x1="55.88" y1="40.64" x2="60.96" y2="40.64" width="0.1524" layer="91"/>
+<wire x1="60.96" y1="40.64" x2="60.96" y2="-15.24" width="0.1524" layer="91"/>
+<pinref part="U$3" gate="G$1" pin="1"/>
+<wire x1="60.96" y1="-15.24" x2="248.92" y2="-15.24" width="0.1524" layer="91"/>
+<wire x1="248.92" y1="-15.24" x2="248.92" y2="-12.7" width="0.1524" layer="91"/>
+</segment>
+</net>
+<net name="N$3" class="0">
+<segment>
+<pinref part="U2" gate="G$1" pin="LED_C"/>
+<wire x1="114.3" y1="40.64" x2="119.38" y2="40.64" width="0.1524" layer="91"/>
+<wire x1="119.38" y1="40.64" x2="119.38" y2="-17.78" width="0.1524" layer="91"/>
+<pinref part="U$3" gate="G$1" pin="3"/>
+<wire x1="119.38" y1="-17.78" x2="251.46" y2="-17.78" width="0.1524" layer="91"/>
+<wire x1="251.46" y1="-17.78" x2="251.46" y2="-12.7" width="0.1524" layer="91"/>
+</segment>
+</net>
+<net name="N$4" class="0">
+<segment>
+<pinref part="U3" gate="G$1" pin="LED_C"/>
+<wire x1="172.72" y1="40.64" x2="180.34" y2="40.64" width="0.1524" layer="91"/>
+<wire x1="180.34" y1="40.64" x2="180.34" y2="-20.32" width="0.1524" layer="91"/>
+<pinref part="U$3" gate="G$1" pin="5"/>
+<wire x1="180.34" y1="-20.32" x2="254" y2="-20.32" width="0.1524" layer="91"/>
+<wire x1="254" y1="-20.32" x2="254" y2="-12.7" width="0.1524" layer="91"/>
+</segment>
+</net>
+<net name="N$5" class="0">
+<segment>
+<pinref part="U4" gate="G$1" pin="LED_C"/>
+<wire x1="228.6" y1="40.64" x2="236.22" y2="40.64" width="0.1524" layer="91"/>
+<wire x1="236.22" y1="40.64" x2="236.22" y2="-22.86" width="0.1524" layer="91"/>
+<pinref part="U$3" gate="G$1" pin="7"/>
+<wire x1="236.22" y1="-22.86" x2="256.54" y2="-22.86" width="0.1524" layer="91"/>
+<wire x1="256.54" y1="-22.86" x2="256.54" y2="-12.7" width="0.1524" layer="91"/>
+</segment>
+</net>
+<net name="N$6" class="0">
+<segment>
+<wire x1="55.88" y1="50.8" x2="68.58" y2="50.8" width="0.1524" layer="91"/>
+<wire x1="68.58" y1="50.8" x2="68.58" y2="5.08" width="0.1524" layer="91"/>
+<pinref part="U$3" gate="G$1" pin="2"/>
+<wire x1="248.92" y1="2.54" x2="248.92" y2="5.08" width="0.1524" layer="91"/>
+<wire x1="248.92" y1="5.08" x2="68.58" y2="5.08" width="0.1524" layer="91"/>
+<pinref part="U1" gate="G$1" pin="LED_A"/>
+</segment>
+</net>
+<net name="N$7" class="0">
+<segment>
+<pinref part="U2" gate="G$1" pin="LED_A"/>
+<wire x1="114.3" y1="50.8" x2="124.46" y2="50.8" width="0.1524" layer="91"/>
+<wire x1="124.46" y1="50.8" x2="124.46" y2="7.62" width="0.1524" layer="91"/>
+<pinref part="U$3" gate="G$1" pin="4"/>
+<wire x1="124.46" y1="7.62" x2="251.46" y2="7.62" width="0.1524" layer="91"/>
+<wire x1="251.46" y1="7.62" x2="251.46" y2="2.54" width="0.1524" layer="91"/>
+</segment>
+</net>
+<net name="N$8" class="0">
+<segment>
+<pinref part="U3" gate="G$1" pin="LED_A"/>
+<wire x1="172.72" y1="50.8" x2="185.42" y2="50.8" width="0.1524" layer="91"/>
+<wire x1="185.42" y1="50.8" x2="185.42" y2="10.16" width="0.1524" layer="91"/>
+<pinref part="U$3" gate="G$1" pin="6"/>
+<wire x1="185.42" y1="10.16" x2="254" y2="10.16" width="0.1524" layer="91"/>
+<wire x1="254" y1="10.16" x2="254" y2="2.54" width="0.1524" layer="91"/>
+</segment>
+</net>
+<net name="N$9" class="0">
+<segment>
+<pinref part="U4" gate="G$1" pin="LED_A"/>
+<pinref part="U$3" gate="G$1" pin="8"/>
+<wire x1="228.6" y1="50.8" x2="256.54" y2="50.8" width="0.1524" layer="91"/>
+<wire x1="256.54" y1="50.8" x2="256.54" y2="2.54" width="0.1524" layer="91"/>
+</segment>
+</net>
+<net name="+3V3" class="0">
+<segment>
+<pinref part="U$1" gate="G$1" pin="P$40"/>
+<pinref part="+3V1" gate="G$1" pin="+3V3"/>
+<wire x1="40.64" y1="292.1" x2="25.4" y2="292.1" width="0.1524" layer="91"/>
+</segment>
+</net>
+<net name="+5V" class="0">
+<segment>
+<pinref part="U$1" gate="G$1" pin="P$2"/>
+<wire x1="-48.26" y1="289.56" x2="-38.1" y2="289.56" width="0.1524" layer="91"/>
+<pinref part="P+6" gate="1" pin="+5V"/>
+</segment>
+</net>
